File: design/MiniPetri.kicad_pcb (KiCad board)
At the start: 2 copper layers, 105.8 x 55 mm, 29 parts, among them J1 MAX7219 8x8 LED Matrix, SW1 Up, SW10 SW_SPST, SW2 Down, SW3 Left, SW4 Right, SW5 Play/Pause, SW6 Toggle, SW7 Reset, SW8 Step forward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

Commit message: finish up
Parts:
- moved D1 0.96 mm to (167.5, 78.5)
Routing:
- net Net-(D1-A): track 22.3 -> 23.2 mm
Changed lines of the file:
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@@
 			(outputformat 1)
 			(mirror no)
-			(drillshape 1)
+			(drillshape 0)
 			(scaleselection 1)
 			(outputdirectory "")
@@
 	(footprint "Diode_THT:D_DO-41_SOD81_P10.16mm_Horizontal"
 		(layer "B.Cu")
-		(at 167.5 77.5 180)
+		(at 167.5 78.46 180)
 		(descr "Diode, DO-41_SOD81 series, Axial, Horizontal, pin pitch=10.16mm, length*diameter=5.2*2.7mm^2, https://www.diodes.com/assets/Package-Files/DO-41-Plastic.pdf")
 		(tags "Diode DO-41_SOD81 series Axial Horizontal pin pitch 10.16mm  length 5.2mm diameter 2.7mm")
@@
 	(segment
 		(start 157.34 66.159999)
-		(end 157.34 77.5)
+		(end 157.34 78.46)
 		(width 1.5)
 		(layer "B.Cu")

Commit message: add firmware
Parts:
- C2: value 100uF -> 150uF
Connections:
- J1 pad 1: Net-(J1-Pin_1) -> /clk
- J1 pad 2: Net-(J1-Pin_2) -> /cs
- J1 pad 3: Net-(J1-Pin_3) -> /din
- U1 pad 1: Net-(J1-Pin_3) -> R1b
- U1 pad 10: R2b -> /cs
- U1 pad 11: R3b -> /din
- U1 pad 2: Net-(J1-Pin_2) -> R2b
- U1 pad 3: Net-(J1-Pin_1) -> R3b
- U1 pad 9: R1b -> /clk
Routing:
- net Net-(J1-Pin_1): track 97.1 -> 0.00 mm
- net Net-(J1-Pin_2): track 93.4 -> 0.00 mm
- net Net-(J1-Pin_3): track 92.5 -> 0.00 mm
- net /cs: track 0.00 -> 88.1 mm
- net /din: track 0.00 -> 80.0 mm
- net /clk: track 0.00 -> 72.0 mm
- net R1b: track 33.8 -> 44.5 mm
- net R3b: track 40.9 -> 49.9 mm
- net Net-(D70-A): track 31.3 -> 22.6 mm
- net R2b: track 48.4 -> 40.8 mm
- net Net-(D66-A): track 38.2 -> 33.9 mm
