File: design/MiniPetri.kicad_sch (KiCad schematic)
At the start: 29 parts, among them J1 MAX7219 8x8 LED Matrix, SW1 Up, SW10 SW_SPST, SW2 Down, SW3 Left, SW4 Right, SW5 Play/Pause, SW6 Toggle, SW7 Reset, SW8 Step forward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

Commit message: finish up
Parts:
- C2: value 100uF -> 150uF
Changed lines of the file:
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@@
 			)
 		)
-		(property "Value" "100uF"
+		(property "Value" "150uF"
 			(at 36.83 37.846 0)
 			(effects

Commit message: add firmware
Connections:
- net R1b: now also U1.1 (GPIO26/ADC0/A0); no longer U1.9 (GPIO2/SCK)
- net R2b: now also U1.2 (GPIO27/ADC1/A1); no longer U1.10 (GPIO4/MISO)
- net R3b: now also U1.3 (GPIO28/ADC2/A2); no longer U1.11 (GPIO3/MOSI)
- net din: now reaches J1.3 (Pin_3)
- net din: now also U1.11 (GPIO3/MOSI); no longer U1.1 (GPIO26/ADC0/A0)
- net cs: now reaches J1.2 (Pin_2)
- net cs: now also U1.10 (GPIO4/MISO); no longer U1.2 (GPIO27/ADC1/A1)
- net clk: now reaches J1.1 (Pin_1)
- net clk: now also U1.9 (GPIO2/SCK); no longer U1.3 (GPIO28/ADC2/A2)
Other:
- note added: "clk cs din gnd vcc"
- note removed: "vcc gnd din cs clk"
- moved on the sheet: J1
